File: Akira_board.sch (KiCad schematic (older format))
At the start: 37 parts, among them J1 AVR-ISP-6, J2 USB_C_Receptacle_USB2.0, J3 Conn_01x04, J5 Conn_02x04_Odd_Even, SW1 Reset SW, SW2 Boot SW, U1 ATMEGA328P-PU-ND, Y1 16MHz

Commit message: adding sensor directly
Parts:
- J1: symbol Connector:AVR-ISP-6 -> Akira_board-rescue:AVR-ISP-6-Connector
Other:
- note removed: "MAKE SURE TO ADD PINS FOR MOUSE SENSOR"
Changed lines of the file:
@@
 EESchema Schematic File Version 4
-LIBS:Akira_board-cache
 EELAYER 30 0
 EELAYER END
@@
 	2300 2450 2450 2450
 $Comp
-L Connector:AVR-ISP-6 J1
+L Akira_board-rescue:AVR-ISP-6-Connector J1
 U 1 1 63DFD37A
 P 5050 10450
@@
 	1    0    0    -1
 $EndComp
-Text Notes 1150 6000 0    394  ~ 0
-MAKE SURE TO ADD PINS FOR MOUSE SENSOR
 Text Notes 7450 9400 0    50   ~ 0
 Trackball Pins
