File: Akira_board.kicad_pcb (KiCad board)
At the start: 2 copper layers, 110 x 94 mm, 44 parts, among them J1 AVR-ISP-6, J2 USB_C_Receptacle_USB2.0, J3 Conn_01x04, J5 Conn_02x04_Odd_Even, SW1 Reset SW, SW2 Boot SW, U1 ATMEGA328P-PU-ND, Y1 16MHz

Commit message: Before PCB layout
Parts:
- removed D4: LED, LED_THT:LED_D3.0mm_Clear
- removed J3: Conn_01x04, Connector_PinHeader_2.54mm:PinHeader_1x04_P2.54mm_Vertical
- removed J5: Conn_02x04_Odd_Even, Encoder_Ring:ADNS-9800
- removed R2: 1K, Resistor_THT:R_Axial_DIN0207_L6.3mm_D2.5mm_P7.62mm_Horizontal
- removed REF**: Mouse_Pad, Encoder_Ring:Mouse_Pad
- removed REF** (x4): Akira_Board_standoff, Encoder_Ring:Akira_Board_standoff
- removed REF**: ADNS9800, Encoder_Ring:ADNS9800
- removed ~: ~, Encoder_Ring:Lines
- added C10: 4.7uF, Capacitor_THT:C_Rect_L4.0mm_W2.5mm_P2.50mm, F.Cu at (278.7, 116.8)
- added C11: 100nF, Capacitor_THT:C_Disc_D3.8mm_W2.6mm_P2.50mm, F.Cu at (273.4, 117.3)
- added C6: 100nF, Capacitor_THT:C_Disc_D3.8mm_W2.6mm_P2.50mm, F.Cu at (229.0, 87.0)
- added C7: 1uF, Capacitor_THT:C_Rect_L4.0mm_W2.5mm_P2.50mm, F.Cu at (229.2, 106.0)
- added C8: 100nF, Capacitor_THT:C_Disc_D3.8mm_W2.6mm_P2.50mm, F.Cu at (229.0, 100.0)
- added C9: 100nF, Capacitor_THT:C_Disc_D3.8mm_W2.6mm_P2.50mm, F.Cu at (229.0, 93.5)
- added OLED1: ~, Connector_PinHeader_2.54mm:PinHeader_1x04_P2.54mm_Vertical, F.Cu at (-82.0, -10.1)
- added R1_6: 10k, Resistor_THT:R_Axial_DIN0207_L6.3mm_D2.5mm_P7.62mm_Horizontal, F.Cu at (273.9, 98.8)
- added R1_7: 39R, Resistor_THT:R_Axial_DIN0207_L6.3mm_D2.5mm_P7.62mm_Horizontal, F.Cu at (273.9, 105.3)
- added R1_8: 10k, Resistor_THT:R_Axial_DIN0207_L6.3mm_D2.5mm_P7.62mm_Horizontal, F.Cu at (273.9, 111.8)
- added R3: 37.4K, Resistor_THT:R_Axial_DIN0207_L6.3mm_D2.5mm_P7.62mm_Horizontal, F.Cu at (226.7, 112.5)
- added R4: 63.4K, Resistor_THT:R_Axial_DIN0207_L6.3mm_D2.5mm_P7.62mm_Horizontal, F.Cu at (226.9, 118.5)
- added U2: TPS73601DBV, Package_TO_SOT_SMD:SOT-23-5, F.Cu at (230.4, 81.5)
- added U3: ~, AkiraBallParts:PMW3360_1, F.Cu at (277.9, 87.8)
- added U4: SN74LVC1T45DCK, Package_TO_SOT_SMD:SOT-363_SC-70-6, F.Cu at (249.1, 93.4)
- added U5: SN74LVC1T45DCK, Package_TO_SOT_SMD:SOT-363_SC-70-6, F.Cu at (249.1, 97.3)
- added U6: SN74LVC1T45DCK, Package_TO_SOT_SMD:SOT-363_SC-70-6, F.Cu at (249.1, 101.3)
- added U7: SN74LVC1T45DCK, Package_TO_SOT_SMD:SOT-363_SC-70-6, F.Cu at (249.1, 105.2)
- C1, C2: value 20p -> 22p; footprint Capacitor_THT:C_Disc_D5.0mm_W2.5mm_P5.00mm -> Capacitor_THT:C_Rect_L4.0mm_W2.5mm_P2.50mm
- C3: value 4.7u -> 4.7uF; footprint Capacitor_THT:CP_Radial_D4.0mm_P2.00mm -> Capacitor_THT:C_Rect_L4.0mm_W2.5mm_P2.50mm
- C4, C5: value 100n -> 100nF; footprint Capacitor_THT:C_Disc_D5.0mm_W2.5mm_P5.00mm -> Capacitor_THT:C_Disc_D3.8mm_W2.6mm_P2.50mm
- D1, D2, D_I_1, D_I_2, D_I_3, D_I_4, D_I_5: footprint Keebio-Parts:Diode -> Diode_THT:D_DO-35_SOD27_P7.62mm_Horizontal
- F1: footprint Fuse:Fuse_Bourns_MF-RG400 -> Fuse:Fuse_Bourns_MF-RG300
- SW_M_1_1, SW_M_1_2, SW_M_2_1, SW_M_2_2: footprint Encoder_Ring:GM8.0 -> AkiraBallParts:GM8.0
- SW_R_1: footprint Encoder_Ring:Encoder_Ring -> AkiraBallParts:Encoder_Ring
- SW_V_1: footprint Keebio-Parts:RotaryEncoder_EC11 -> Rotary_Encoder:RotaryEncoder_Alps_EC11E-Switch_Vertical_H20mm
- moved R2_1 260.2 mm to (-85.3, 3.50), turned to 0 degrees
- moved R2_2 258.7 mm to (-85.3, 7.55), turned to 0 degrees
- moved D_I_5 195.7 mm to (21.2, 192.7), turned to 0 degrees
- moved D_I_3 189.5 mm to (21.2, 185.6), turned to 0 degrees
- moved D_I_4 188.4 mm to (21.2, 189.1), turned to 0 degrees
- moved D_I_2 185.4 mm to (21.2, 182.0), turned to 0 degrees
- moved D_I_1 178.9 mm to (21.2, 178.4), turned to 0 degrees
- moved SW_M_1_2 172.0 mm to (25.4, 158.0), turned to 0 degrees
- moved SW_M_2_2 166.4 mm to (25.4, 172.1), turned to 0 degrees
- moved R1 164.5 mm to (60.4, -51.8), turned to 0 degrees
- moved SW1 158.9 mm to (60.8, -62.2)
- moved R1_5 157.6 mm to (17.9, 48.5), turned to 0 degrees
- moved SW2 144.5 mm to (72.0, -62.0)
- moved J1 124.0 mm to (155.0, -72.5), turned to 0 degrees
- moved F1 119.3 mm to (18.9, 85.4), turned to 0 degrees
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Connections:
- net MI renamed MISO
- net MO renamed MOSI
- net SC renamed SCK
- J2 pad A8: Net-(J2-PadA8) -> unconnected-(J2-SBU1-PadA8)
- J2 pad B8: Net-(J2-PadB8) -> unconnected-(J2-SBU2-PadB8)
- SW_M_1_1 pad NC: Net-(SW_M_1_1-PadNC) -> unconnected-(SW_M_1_1-PadNC)
- SW_M_1_2 pad NC: Net-(SW_M_1_2-PadNC) -> unconnected-(SW_M_1_2-PadNC)
- SW_M_2_1 pad NC: Net-(SW_M_2_1-PadNC) -> unconnected-(SW_M_2_1-PadNC)
- SW_M_2_2 pad NC: Net-(SW_M_2_2-PadNC) -> unconnected-(SW_M_2_2-PadNC)
- U1 pad 16: SS -> NCS
- U1 pad 21: Net-(U1-Pad21) -> unconnected-(U1-AREF-Pad21)
- U1 pad 24: Net-(U1-Pad24) -> unconnected-(U1-PC1-Pad24)
- U1 pad 3: Net-(U1-Pad3) -> unconnected-(U1-PD1-Pad3)
- U1 pad 6: MOT -> MOTION
Routing:
- net GND: track 267.5 -> 0.00 mm, vias 3 -> 0
- net MOSI: track 237.5 -> 0.00 mm, vias 4 -> 0
- net MISO: track 215.1 -> 0.00 mm, vias 6 -> 0
- net SCK: track 187.6 -> 0.00 mm, vias 4 -> 0
- net VK_B: track 175.7 -> 0.00 mm, vias 4 -> 0
- net +5V: track 169.8 -> 0.00 mm, vias 4 -> 0
- net D+: track 161.4 -> 0.00 mm, vias 3 -> 0
- net D-: track 158.2 -> 0.00 mm, vias 3 -> 0
- net COL0: track 144.2 -> 0.00 mm, vias 1 -> 0
- net SS: track 143.6 -> 0.00 mm, vias 2 -> 0
- net Net-(D_I_1-A): track 141.8 -> 0.00 mm, vias 1 -> 0
- net Net-(D_I_3-A): track 140.1 -> 0.00 mm, vias 2 -> 0
- net Net-(D_I_2-A): track 133.3 -> 0.00 mm, vias 2 -> 0
- net RING_A: track 128.9 -> 0.00 mm, vias 1 -> 0
- net I2C_SDA: track 128.2 -> 0.00 mm, vias 5 -> 0
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Other:
- board outline removed
- net class Default removed
- board text removed: "A-C-B"
- board text removed: "B-C-A"
- board text removed: "JLCJLCJLCJLC"

Commit message: reduced files
Parts:
- moved SW_R_1 108.4 mm to (150.0, 100.0)
Changed lines of the file:
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@@
 	(footprint "AkiraBallParts:Encoder_Ring"
 		(layer "F.Cu")
-		(at 139.44 -7.91)
+		(at 150 100)
 		(property "Reference" "SW_R_1"
 			(at 0.825 -1.925 0)
@@
 		)
 	)
+	(gr_line
+		(start 200 150)
+		(end 100 50)
+		(stroke
+			(width 0.1)
+			(type default)
+		)
+		(layer "Eco2.User")
+	)
+	(gr_line
+		(start 200 50)
+		(end 100 150)
+		(stroke
+			(width 0.1)
+			(type default)
+		)
+		(layer "Eco2.User")
+	)
+	(gr_rect
+		(start 100 50)
+		(end 200 150)
+		(stroke
+			(width 0.1)
+			(type default)
+		)
+		(fill none)
+		(layer "Eco2.User")
+	)
 )

Commit message: nice corners designed
Parts:
- C3: footprint Capacitor_THT:C_Rect_L4.0mm_W2.5mm_P2.50mm -> Capacitor_THT:CP_Radial_D4.0mm_P1.50mm
- OLED1: footprint Connector_PinHeader_2.54mm:PinHeader_1x04_P2.54mm_Vertical -> AkiraBallParts:OLED_PinHeader_1x04_P2.54mm
- U1: footprint Package_DIP:DIP-28_W7.62mm_Socket -> AkiraBallParts:DIP-28_AtMega328PU
- U3: moved to B.Cu
- Y1: footprint Crystal:Crystal_HC49-U_Vertical -> Crystal:Crystal_HC49-4H_Vertical
- moved OLED1 219.3 mm to (108.8, 98.1), turned to -90 degrees
- moved R2_1 215.7 mm to (115.3, 82.8), turned to -26.25 degrees
- moved R2_2 214.2 mm to (113.6, 86.8), turned to -20 degrees
- moved J1 179.7 mm to (198.7, 101.8)
- moved SW_M_2_2 175.4 mm to (196.6, 133.6), turned to 135 degrees
- moved C3 168.7 mm to (176.3, 80.7), turned to -55 degrees
- moved SW_M_2_1 167.6 mm to (191.0, 139.0), turned to 135 degrees
- moved C4 164.5 mm to (177.1, 73.0), turned to -135 degrees
- moved C5 160.4 mm to (173.8, 76.3), turned to -135 degrees
- moved J2 158.4 mm to (176.3, 54.1)
- moved D1 157.2 mm to (174.5, 70.0), turned to -130 degrees
- moved D_I_1 156.6 mm to (130.6, 66.5), turned to -60 degrees
- moved D_I_2 155.9 mm to (127.8, 68.3), turned to -55 degrees
- moved F1 155.7 mm to (171.9, 56.2), turned to 180 degrees
- moved D_I_3 155.2 mm to (125.2, 70.3), turned to -50 degrees
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Other:
- board outline added: 110 x 94 mm
- board text added: "Buttons"
- board text added: "OLED"
- board text added: "Power Caps"
- board text added: "Power Reg"
- board text added: "Rotary_Encoder"
- board text added: "SW"
- board text added: "SW_R_1"
- board text added: "USB Circuit"

Commit message: Before routing PCB
Parts:
- added H1: MountingHole_Pad, AkiraBallParts:M2 Mounting Hole, F.Cu at (108.0, 57.0)
- added H2: MountingHole_Pad, AkiraBallParts:M2 Mounting Hole, F.Cu at (192.0, 57.0)
- added H3: MountingHole_Pad, AkiraBallParts:M2 Mounting Hole, F.Cu at (201.0, 104.0)
- added H4: MountingHole_Pad, AkiraBallParts:M2 Mounting Hole, F.Cu at (150.0, 133.5)
- added H5: MountingHole_Pad, AkiraBallParts:M2 Mounting Hole, F.Cu at (99.0, 104.0)
- added H6: MountingHole_Pad, AkiraBallParts:M2 Mounting Hole, F.Cu at (122.5, 119.5)
- added H7: MountingHole_Pad, AkiraBallParts:M2 Mounting Hole, F.Cu at (177.5, 119.5)
- moved J1 94.4 mm to (114.5, 59.0), turned to 90 degrees
- moved SW1 79.7 mm to (158.0, 115.8), turned to 180 degrees
- moved SW2 68.4 mm to (148.5, 115.8), turned to 180 degrees
- moved SW_V_1 6.66 mm to (112.0, 107.0)
