File: Akira_board.kicad_pcb (KiCad board)
At the start: 2 copper layers, 110 x 94 mm, 58 parts, among them J1 AVR-ISP-6, J2 USB_C_Receptacle_USB2.0, SW1 Reset SW, SW2 Boot SW, U1 ATMEGA328P-PU-ND, U2 TPS73601DBV, U4 SN74LVC1T45DCK, U5 SN74LVC1T45DCK, U6 SN74LVC1T45DCK, U7 SN74LVC1T45DCK, Y1 16MHz

Commit message: Dump
Parts:
- ISP1: renamed from J1; footprint Connector_PinHeader_2.54mm:PinHeader_2x03_P2.54mm_Vertical -> AkiraBallParts:SKEDD_6PinConnectingHole
- moved C2 15.8 mm to (185.2, 92.8)
- moved C1 15.8 mm to (185.2, 77.2)
- moved F1 12.4 mm to (182.8, 62.2), turned to 0 degrees
- moved USB1 8.04 mm to (182.6, 59.1), turned to 180 degrees
- moved R1_3 7.69 mm to (159.0, 66.2), turned to 75 degrees
- moved R2_1 7.66 mm to (122.1, 86.3), turned to 153.75 degrees
- moved R1_8 7.62 mm to (192.5, 103.7), turned to 175 degrees
- moved R1_6 7.62 mm to (191.2, 111.1), turned to 165 degrees
- moved R1_7 7.62 mm to (192.1, 107.4), turned to 170 degrees
- moved D_I_4 6.75 mm to (127.8, 68.3), turned to -55 degrees
- moved ISP1 5.01 mm to (119.2, 57.2), turned to 0 degrees
- moved D_I_3 3.38 mm to (122.7, 72.6), turned to -45 degrees
- moved D_I_2 3.34 mm to (125.2, 70.4), turned to -50 degrees
- moved C9 2.54 mm to (143.2, 60.8), turned to 100 degrees
- moved C6 2.48 mm to (148.3, 60.2), turned to 92.5 degrees
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- renumbered U1 to ATMEGA328P1, SW_V_1 to KNOB1, U4 to LS1, U5 to LS2, U6 to LS3, U7 to LS4, U3 to PMW3360, SW_R_1 to SCROLL_RING1, J2 to USB1, U2 to VR1
Connections:
- net Net-(U1-PB6) renamed CRYSTAL-
- net Net-(U1-PB7) renamed CRYSTAL+
Routing:
- net I2C_SDA: track 0.00 -> 196.3 mm, vias 0 -> 4
- net I2C_SCL: track 0.00 -> 195.1 mm, vias 0 -> 4
- net +5V: track 0.00 -> 182.8 mm, vias 0 -> 3
- net RESET: track 0.00 -> 165.5 mm, vias 0 -> 6
- net NCS: track 0.00 -> 141.4 mm, vias 0 -> 7
- net VDD: track 0.00 -> 135.2 mm, vias 0 -> 3
- net PMW.MISO: track 0.00 -> 134.2 mm, vias 0 -> 3
- net MOSI: track 0.00 -> 129.9 mm, vias 0 -> 8
- net MISO: track 0.00 -> 128.9 mm, vias 0 -> 4
- net Net-(D_I_5-A): track 0.00 -> 118.6 mm, vias 0 -> 3
- net COL0: track 0.00 -> 116.1 mm, vias 0 -> 4
- net GND: track 0.00 -> 113.2 mm, vias 0 -> 21
- net Net-(D_I_3-A): track 0.00 -> 112.3 mm, vias 0 -> 7
- net ROW2: track 0.00 -> 106.3 mm, vias 0 -> 4
- net SCK: track 0.00 -> 105.0 mm, vias 0 -> 4
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- added copper zone on F.Cu, net GND
Other:
- rule pad_to_mask_clearance: 0.051 -> 0
- board text added: "5V|MOSI|GND MISO|SCK|Reset"
- board text added: "Akira Ball : Rev 2 By : Kye Morris-Takamoto MoonShine Studio JLCJLCJLCJLC"
- board text added: "SDA|SCL 5V|GND"
- board text removed: "SW_R_1"

Commit message: Save
Parts:
- moved SW_M_2_2 1.29 mm to (197.4, 132.6)
- moved SW_M_2_1 0.55 mm to (190.6, 139.4)
- moved SW_M_1_1 0.27 mm to (103.6, 131.8)
Routing:
- net COL1: track 64.8 -> 74.3 mm
- net Net-(D_I_5-A): track 118.6 -> 119.9 mm
- net COL0: track 116.1 -> 115.6 mm

Commit message: Before PCB Fix
Parts:
- PMW3360: footprint AkiraBallParts:PMW3360_1 -> Akira_Ball_Parts:PMW3360_2
Connections:
- ATMEGA328P1 pad 24: unconnected-(ATMEGA328P1-PC1-Pad24) -> VK_A
- KNOB1 pad A: RING_A -> VK_A
- LS3 pad 5: NCS -> +5V
Routing:
- net VK_A: track 0.00 -> 120.9 mm, vias 0 -> 8
- net RING_A: track 70.0 -> 41.2 mm
- net NCS: track 141.4 -> 126.0 mm
- net Net-(PMW3360-VDDPIX): track 36.2 -> 33.6 mm
- net +5V: track 182.8 -> 185.0 mm
- net PMW.SCK: track 44.4 -> 46.5 mm
- net PMW.MOSI: track 44.5 -> 46.5 mm
- net PMW.MISO: track 134.2 -> 136.2 mm
- net PMW.NCS: track 40.6 -> 42.7 mm
- net VDD: track 135.2 -> 136.2 mm
- net Net-(PMW3360-NRESET): track 31.1 -> 30.2 mm
- net Net-(PMW3360-LED_P): track 94.4 -> 95.2 mm

Commit message: Save for now
Parts:
- removed C3: 4.7uF, Capacitor_THT:CP_Radial_D4.0mm_P1.50mm
- removed SW1: Reset SW, Button_Switch_THT:SW_PUSH_6mm
- removed SW2: Boot SW, Button_Switch_THT:SW_PUSH_6mm
- removed Y1: 16MHz, Crystal:Crystal_HC49-4H_Vertical
- added C12: 4.7uF, Capacitor_SMD:C_0805_2012Metric, F.Cu at (219.2, 47.5)
- added R1_10: 2R, Resistor_SMD:R_0603_1608Metric, F.Cu at (214.9, 51.8)
- added R1_11: 2R, Resistor_SMD:R_0603_1608Metric, F.Cu at (214.9, 54.3)
- added R1_12: 20R, Resistor_SMD:R_0603_1608Metric, F.Cu at (214.9, 56.8)
- added R1_13: 20R, Resistor_SMD:R_0603_1608Metric, F.Cu at (214.9, 59.3)
- added R1_9: 2R, Resistor_SMD:R_0603_1608Metric, F.Cu at (214.9, 49.3)
- added R2: 7.5K, Resistor_SMD:R_0603_1608Metric, F.Cu at (214.9, 44.3)
- added R5: 7.5K, Resistor_SMD:R_0603_1608Metric, F.Cu at (214.9, 46.8)
- added U1: ~, Akira_Ball_Parts:Switch SMD-4P,5.1x5.1mm, F.Cu at (144.2, 118.4)
- added U2: ~, Akira_Ball_Parts:Switch SMD-4P,5.1x5.1mm, F.Cu at (154.0, 118.6)
- added Y2: Crystal_GND24, Crystal:Crystal_SMD_3225-4Pin_3.2x2.5mm, F.Cu at (219.6, 51.3)
- C1, C2: value 22p -> 12p; footprint Capacitor_THT:C_Rect_L4.0mm_W2.5mm_P2.50mm -> Capacitor_SMD:C_0603_1608Metric
- C10: footprint Capacitor_THT:C_Rect_L4.0mm_W2.5mm_P2.50mm -> Capacitor_SMD:C_0805_2012Metric
- C11, C4, C5, C6, C8, C9: footprint Capacitor_THT:C_Disc_D3.8mm_W2.6mm_P2.50mm -> Capacitor_SMD:C_0603_1608Metric
- C7: footprint Capacitor_THT:C_Rect_L4.0mm_W2.5mm_P2.50mm -> Capacitor_SMD:C_0603_1608Metric
- D1, D2, D_I_1, D_I_2, D_I_3, D_I_4, D_I_5: footprint Diode_THT:D_DO-35_SOD27_P7.62mm_Horizontal -> Diode_SMD:D_SOD-123
- F1: footprint Fuse:Fuse_Bourns_MF-RG300 -> Fuse:Fuse_0805_2012Metric
- R1, R1_1, R1_2, R1_5, R1_6, R1_8, R2_1, R2_2: footprint Resistor_THT:R_Axial_DIN0207_L6.3mm_D2.5mm_P7.62mm_Horizontal -> Resistor_SMD:R_0603_1608Metric
- R1_3, R1_4: value 75R -> 47R; footprint Resistor_THT:R_Axial_DIN0207_L6.3mm_D2.5mm_P7.62mm_Horizontal -> Resistor_SMD:R_0603_1608Metric
- R1_7: value 39R -> 33R; footprint Resistor_THT:R_Axial_DIN0207_L6.3mm_D2.5mm_P7.62mm_Horizontal -> Resistor_SMD:R_0603_1608Metric
- R3: value 37.4K -> 30K; footprint Resistor_THT:R_Axial_DIN0207_L6.3mm_D2.5mm_P7.62mm_Horizontal -> Resistor_SMD:R_0603_1608Metric
- R4: value 63.4K -> 56K; footprint Resistor_THT:R_Axial_DIN0207_L6.3mm_D2.5mm_P7.62mm_Horizontal -> Resistor_SMD:R_0603_1608Metric
- SW_M_1_1, SW_M_1_2, SW_M_2_1, SW_M_2_2: footprint AkiraBallParts:GM8.0 -> Akira_Ball_Parts:GM8.0
- moved SW_M_2_1 130.9 mm to (81.0, 67.9), turned to 0 degrees
- moved SW_M_2_2 129.9 mm to (81.0, 74.9), turned to 0 degrees
- moved SW_M_1_2 85.8 mm to (80.9, 58.0), turned to 0 degrees
- moved SW_M_1_1 83.9 mm to (80.9, 51.0), turned to 0 degrees
- moved C10 82.8 mm to (219.2, 44.5), turned to 0 degrees
Connections:
- C10 pad 1: Net-(PMW3360-VDDPIX) -> +5V
- R1_3 pad 1: D- -> Net-(R1_13-Pad2)
- R1_4 pad 2: D+ -> Net-(R1_12-Pad1)
- R1_7 pad 1: VDD -> Net-(R1_7-Pad1)
- R3 pad 2: Net-(VR1-FB) -> Net-(R2-Pad1)
- R4 pad 2: GND -> Net-(R4-Pad2)
Routing:
- net I2C_SDA: track 196.6 -> 0.00 mm, vias 4 -> 0
- net I2C_SCL: track 195.5 -> 0.00 mm, vias 4 -> 0
- net +5V: track 185.0 -> 0.00 mm, vias 3 -> 0
- net RESET: track 165.5 -> 0.00 mm, vias 6 -> 0
- net VDD: track 136.2 -> 0.00 mm, vias 3 -> 0
- net PMW.MISO: track 136.2 -> 0.00 mm, vias 3 -> 0
- net MOSI: track 129.9 -> 0.00 mm, vias 8 -> 0
- net MISO: track 128.9 -> 0.00 mm, vias 4 -> 0
- net NCS: track 126.0 -> 0.00 mm, vias 7 -> 0
- net VK_A: track 120.9 -> 0.00 mm, vias 8 -> 0
- net Net-(D_I_5-A): track 119.9 -> 0.00 mm, vias 3 -> 0
- net COL0: track 115.6 -> 0.00 mm, vias 4 -> 0
- net GND: track 113.2 -> 0.00 mm, vias 21 -> 0
- net Net-(D_I_3-A): track 112.1 -> 0.00 mm, vias 7 -> 0
- net ROW2: track 106.3 -> 0.00 mm, vias 4 -> 0
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- removed copper zone on F.Cu, net GND
Other:
- board text removed: "Rotary_Encoder"

Commit message: save for now
Parts:
- moved SW_M_2_1 130.4 mm to (190.5, 138.8), turned to 135 degrees
- moved SW_M_2_2 129.3 mm to (196.8, 132.5), turned to 135 degrees
- moved SW_M_1_1 92.4 mm to (109.3, 138.9), turned to 45 degrees
- moved SW_M_1_2 77.8 mm to (103.1, 132.7), turned to 45 degrees
- moved D_I_3 61.6 mm to (167.2, 30.0), turned to 0 degrees
- moved D_I_2 61.0 mm to (167.0, 26.0), turned to 0 degrees
- moved C11 59.7 mm to (222.0, 67.5), turned to 0 degrees
- moved D_I_5 59.6 mm to (167.0, 38.0), turned to 0 degrees
- moved D_I_1 57.5 mm to (167.0, 22.0), turned to 0 degrees
- moved R1_12 57.0 mm to (158.0, 58.0)
- moved R1_13 56.7 mm to (158.3, 62.0)
- moved R2_1 55.6 mm to (154.0, 40.8), turned to 0 degrees
- moved R1_6 54.2 mm to (226.0, 69.5), turned to 0 degrees
- moved LS4 53.8 mm to (156.1, 35.4), turned to 0 degrees
- moved R2_2 53.4 mm to (147.4, 45.4), turned to 0 degrees
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Other:
- board text added: "Crystal"

Commit message: SMT (done hopefully)
Parts:
- added H8: , , F.Cu at (138.0, 100.0)
- added H9: , , F.Cu at (162.0, 100.0)
- added R6: 10K, Resistor_SMD:R_0603_1608Metric, F.Cu at (115.8, 90.8)
- KNOB1: footprint Rotary_Encoder:RotaryEncoder_Alps_EC11E-Switch_Vertical_H20mm -> Akira_Ball_Parts:RotaryEncoder_Alps_EC11E-Switch_Vertical_H20mm
- U1, U2: value ~ -> SW
- USB1: footprint Connector_USB:USB_C_Receptacle_GCT_USB4085 -> Akira_Ball_Parts:USB_C_16P_SMD_C3025063
- moved R1_8 103.4 mm to (122.8, 72.6), turned to -45 degrees
- moved R1_6 101.2 mm to (125.0, 74.9), turned to -45 degrees
- moved C12 96.7 mm to (125.3, 70.5), turned to 130 degrees
- moved C11 92.8 mm to (129.6, 75.7), turned to -50 degrees
- moved R1_7 91.7 mm to (128.0, 68.5), turned to 125 degrees
- moved R1_9 88.0 mm to (129.7, 71.0), turned to 125 degrees
- moved R1_10 85.5 mm to (130.7, 66.7), turned to -60 degrees
- moved R1_11 84.0 mm to (132.3, 69.2), turned to -60 degrees
- moved D_I_2 74.2 mm to (117.5, 81.2), turned to 150 degrees
- moved D_I_5 71.8 mm to (114.7, 87.2), turned to 160 degrees
- moved D_I_4 71.6 mm to (115.9, 84.1), turned to 155 degrees
- moved D_I_1 70.7 mm to (121.2, 75.8), turned to 140 degrees
- moved D_I_3 68.2 mm to (119.2, 78.5), turned to 145 degrees
- moved R2_1 67.2 mm to (112.0, 93.3), turned to -10 degrees
- moved R5 64.4 mm to (153.1, 64.7), turned to -95 degrees
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Routing:
- net +5V: track 0.00 -> 225.4 mm, vias 0 -> 4
- net ROW2: track 0.00 -> 212.9 mm, vias 0 -> 7
- net I2C_SDA: track 0.00 -> 209.6 mm, vias 0 -> 3
- net I2C_SCL: track 0.00 -> 208.0 mm, vias 0 -> 6
- net ROW1: track 0.00 -> 206.4 mm, vias 0 -> 3
- net RESET: track 0.00 -> 201.2 mm, vias 0 -> 6
- net VK_B: track 0.00 -> 188.7 mm, vias 0 -> 2
- net VK_A: track 0.00 -> 182.4 mm, vias 0 -> 2
- net ROW0: track 0.00 -> 180.7 mm, vias 0 -> 3
- net Net-(D_I_3-A): track 0.00 -> 169.4 mm, vias 0 -> 4
- net COL0: track 0.00 -> 166.7 mm, vias 0 -> 1
- net Net-(D_I_5-A): track 0.00 -> 165.3 mm, vias 0 -> 2
- net VDD: track 0.00 -> 151.9 mm, vias 0 -> 4
- net COL1: track 0.00 -> 148.0 mm, vias 0 -> 1
- net MISO: track 0.00 -> 133.7 mm, vias 0 -> 6
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- added copper zone on B.Cu, net GND
- added copper zone on F.Cu, net GND
Other:
- board text added: "Akira Ball : Rev 2 By : Kye Morris-Takamoto rolling_ball Lab"
- board text added: "Level Shifter"
- board text added: "PWM3360 Extras"
- board text removed: "Akira Ball : Rev 2 By : Kye Morris-Takamoto MoonShine Studio JLCJLCJLCJLC"
