File: Akira_board.kicad_sch (KiCad schematic)
At the start: 44 parts, among them J1 AVR-ISP-6, J2 USB_C_Receptacle_USB2.0, J3 Conn_01x04, J5 Conn_02x04_Odd_Even, SW1 Reset SW, SW2 Boot SW, U1 ATMEGA328P-PU-ND, U2 TPS73601DBV, Y1 16MHz

Commit message: Before PCB layout
Parts:
- removed D4: LED, LED_THT:LED_D3.0mm_Clear, symbol Device:LED
- removed J3: Conn_01x04, Connector_PinHeader_2.54mm:PinHeader_1x04_P2.54mm_Vertical, symbol Akira_board-rescue:Conn_01x04_Female-Connector
- removed J5: Conn_02x04_Odd_Even, Encoder_Ring:ADNS-9800, symbol Connector_Generic:Conn_02x04_Odd_Even
- removed R2: 1K, Resistor_THT:R_Axial_DIN0207_L6.3mm_D2.5mm_P7.62mm_Horizontal, symbol Device:R
- added C10: 4.7uF, Capacitor_THT:C_Rect_L4.0mm_W2.5mm_P2.50mm, symbol Akira_board-rescue:CP1-Device
- added C11: 100nF, Capacitor_THT:C_Disc_D3.8mm_W2.6mm_P2.50mm, symbol Device:C
- added OLED1: ~, Connector_PinHeader_2.54mm:PinHeader_1x04_P2.54mm_Vertical, symbol Akira_board-rescue:OLED_display_128x32
- added R1_6, R1_8: 10k, Resistor_THT:R_Axial_DIN0207_L6.3mm_D2.5mm_P7.62mm_Horizontal, symbol Device:R
- added R1_7: 39R, Resistor_THT:R_Axial_DIN0207_L6.3mm_D2.5mm_P7.62mm_Horizontal, symbol Device:R
- added U3: ~, AkiraBallParts:PMW3360_1, symbol Akira_board-rescue:PMW3350
- added U4, U5, U6, U7: SN74LVC1T45DCK, Package_TO_SOT_SMD:SOT-363_SC-70-6, symbol Logic_LevelTranslator:SN74LVC1T45DCK
- C1, C2: value 20p -> 22p; footprint Capacitor_THT:C_Disc_D5.0mm_W2.5mm_P5.00mm -> Capacitor_THT:C_Rect_L4.0mm_W2.5mm_P2.50mm; Digikey# (none) -> BC1005CT-ND; Part Check (none) -> x
- C3: value 4.7u -> 4.7uF; footprint Capacitor_THT:CP_Radial_D4.0mm_P2.00mm -> Capacitor_THT:C_Rect_L4.0mm_W2.5mm_P2.50mm; Digikey# (none) -> 445-FG18X5R1E475KRT00-ND/445-5324-ND; Part Check (none) -> x
- C4, C5: value 100n -> 100nF; footprint Capacitor_THT:C_Disc_D5.0mm_W2.5mm_P5.00mm -> Capacitor_THT:C_Disc_D3.8mm_W2.6mm_P2.50mm; Digikey# (none) -> BC1084CT-ND; Part Check (none) -> x
- C6, C8, C9: footprint (none) -> Capacitor_THT:C_Disc_D3.8mm_W2.6mm_P2.50mm; Digikey# (none) -> BC1084CT-ND; Part Check (none) -> x
- C7: footprint (none) -> Capacitor_THT:C_Rect_L4.0mm_W2.5mm_P2.50mm; Digikey# (none) -> 445-180204-ND; Part Check (none) -> x
- D1, D2: footprint Keebio-Parts:Diode -> Diode_THT:D_DO-35_SOD27_P7.62mm_Horizontal; Digikey# (none) -> BZX79C3V6-ND; Part Check (none) -> x
- D_I_1, D_I_2, D_I_3, D_I_4, D_I_5: footprint Keebio-Parts:Diode -> Diode_THT:D_DO-35_SOD27_P7.62mm_Horizontal; Digikey# (none) -> 4878-1N4148CT-ND; Part Check (none) -> x
- F1: footprint Fuse:Fuse_Bourns_MF-RG400 -> Fuse:Fuse_Bourns_MF-RG300; Digikey# (none) -> 5923-0ZRC0017FF1E-ND; Part Check (none) -> x
- J2: Digikey# (none) -> 2073-USB4085-GF-ACT-ND; Part Check (none) -> x
- R1: Digikey# (none) -> 738-RNMF12FTD10K0CT-ND; Wattage (none) -> 1/2
- R1_1, R1_2: Digikey# (none) -> 13-MFR50SFTE52-5K1CT-ND; Wattage (none) -> 1/2
- R1_3, R1_4: Digikey# (none) -> 13-MFR50SFTE52-75RCT-ND; Wattage (none) -> 1/2
- R1_5: Digikey# (none) -> 13-MFR50SFTE52-1K5CT-ND; Wattage (none) -> 1/2
- R2_1, R2_2: Digikey# (none) -> 13-MFR50SFTE52-4K7CT-ND; Wattage (none) -> 1/2
- R3: footprint (none) -> Resistor_THT:R_Axial_DIN0207_L6.3mm_D2.5mm_P7.62mm_Horizontal; Digikey# (none) -> MFR-25FBF52-37K4; Part Check (none) -> x; Wattage (none) -> 1/4
- R4: footprint (none) -> Resistor_THT:R_Axial_DIN0207_L6.3mm_D2.5mm_P7.62mm_Horizontal; Digikey# (none) -> 13-MFR-25FTE52-63K4CT-ND; Part Check (none) -> x; Wattage (none) -> 1/4
- SW1, SW2: Digikey# (none) -> SW402-ND
- SW_M_1_1, SW_M_1_2, SW_M_2_1, SW_M_2_2: footprint Encoder_Ring:GM8.0 -> AkiraBallParts:GM8.0; Part Check (none) -> x
- SW_R_1: footprint Encoder_Ring:Encoder_Ring -> AkiraBallParts:Encoder_Ring; Digikey# (none) -> 118-PER561-P115-N0015-ND
- SW_V_1: footprint Keebio-Parts:RotaryEncoder_EC11 -> Rotary_Encoder:RotaryEncoder_Alps_EC11E-Switch_Vertical_H20mm; Digikey# (none) -> PEC11R-4220K-S0024-ND
- U1: Digikey# (none) -> ATMEGA328P-PU-ND
- U2: Digikey# (none) -> 296-18255-1-ND
- Y1: Digikey# (none) -> 535-9041-ND
Connections:
- net +5V: now also OLED1.2 (VCC), U4.1 (VCCA), U4.5 (DIR), U5.1 (VCCA), U5.5 (DIR), U6.1 (VCCA), U7.1 (VCCA), U7.5 (DIR)
- net GND: now also C10.2, C11.2, OLED1.1 (GND), U3.8 (GND), U4.2 (GND), U5.2 (GND), U6.2 (GND), U7.2 (GND)
- net I2C_SCL: now also OLED1.3 (SCL)
- net I2C_SDA: now also OLED1.4 (SDA)
- net VDD: now reaches C8.1, C9.1, R3.1, U2.5 (OUT)
- net VDD: now also R1_6.1, R1_7.1, R1_8.1, U3.4 (VDD), U3.5 (VDDIO), U4.6 (VCCB), U5.6 (VCCB), U6.6 (VCCB), U7.6 (VCCB)
- net MI renamed MISO
- net MISO: now also U6.3 (A)
- net MO renamed MOSI
- net MOSI: now also U5.3 (A)
- net MOT renamed MOTION
- net SC renamed SCK
- net SCK: now also U7.3 (A)
- net SS renamed NCS
- net NCS: now also U4.3 (A), U6.5 (DIR)
- new net: R1_6.2, U3.7 (NRESET)
- new net: C10.1, C11.1, U3.3 (VDDPIX)
- new net: R1_7.2, U3.15 (LED_P)
- new net PMW.MISO: R1_8.2, U3.12 (MISO), U6.4 (B)
- new net PMW.MOSI: U3.11 (MOSI), U5.4 (B)
- new net PMW.NCS: U3.13 (NCS), U4.4 (B)
- new net PMW.SCK: U3.10 (SCLK), U7.4 (B)
- no-connect marks 6 -> 12
Other:
- note added: "Buttons & Encoders"
- note added: "Chip Select"
- note added: "Clicks & Volume"
- note added: "Level Shifters"
- note added: "MISO"
- note added: "MOSI"
- note added: "OLED Display"
- note added: "Power Regulator"
- note added: "Scroll Encoder"
- note added: "Serial Clock"
- note added: "not needed?"
- note removed: "I2C Pull Up"
- note removed: "ISP Activity Indicatior"
- note removed: "Inputs"
- note removed: "Left to Right: GND-VCC-SCL-SDA"
- note removed: "MI = MISO MO = MOSI SS = Slave Select / Chip Select SC = SPI Clock MOT = Motion (active low interrupt line) AG = Analog Ground DG = Digital Ground VI = Voltage in up to +6V"
- note removed: "Trackball Pins"
- note removed: "Trackball Voltage Regulator"
- note removed: "[X] ATmega328P circuit [X] Crystal [X] Boot & Reset Button [X] Power noise [X] ISP Activity Indicator [X] ISP Programmer [X] I2C Pull Up [X] USB-C Connector [X] Inputs [X] Trackball Pins"
- moved on the sheet: C1, C2, C3, C4, C5, C6, C7, C8, C9, D1, D2, D_I_1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

Commit message: nice corners designed
Parts:
- added U8: USBLC6-2SC6, Package_TO_SOT_SMD:SOT-23-6, symbol Power_Protection:USBLC6-2SC6
- C3: footprint Capacitor_THT:C_Rect_L4.0mm_W2.5mm_P2.50mm -> Capacitor_THT:CP_Radial_D4.0mm_P1.50mm; Digikey# 445-FG18X5R1E475KRT00-ND/445-5324-ND -> 10-ECE-A1EKS4R7BCT-ND
- OLED1: footprint Connector_PinHeader_2.54mm:PinHeader_1x04_P2.54mm_Vertical -> AkiraBallParts:OLED_PinHeader_1x04_P2.54mm
- U1: footprint Package_DIP:DIP-28_W7.62mm_Socket -> AkiraBallParts:DIP-28_AtMega328PU
- Y1: footprint Crystal:Crystal_HC49-U_Vertical -> Crystal:Crystal_HC49-4H_Vertical
Changed lines of the file:
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@@
 			)
 		)
-		(property "Footprint" "Package_DIP:DIP-28_W7.62mm_Socket"
+		(property "Footprint" "AkiraBallParts:DIP-28_AtMega328PU"
 			(at 80.01 27.94 0)
 			(effects
@@
 			)
 		)
-		(property "Footprint" "Crystal:Crystal_HC49-U_Vertical"
+		(property "Footprint" "Crystal:Crystal_HC49-4H_Vertical"
 			(at 35.56 50.8 0)
 			(effects
@@
 			)
 		)
-		(property "Footprint" "Capacitor_THT:C_Rect_L4.0mm_W2.5mm_P2.50mm"
+		(property "Footprint" "Capacitor_THT:CP_Radial_D4.0mm_P1.50mm"
 			(at 64.77 232.41 0)
 			(effects
@@
 			)
 		)
-		(property "Digikey#" "445-FG18X5R1E475KRT00-ND/445-5324-ND"
+		(property "Digikey#" "10-ECE-A1EKS4R7BCT-ND"
 			(at 64.77 232.41 0)
 			(effects
@@
 	)
 	(symbol
+		(lib_id "Power_Protection:USBLC6-2SC6")
+		(at -39.37 107.95 0)
+		(unit 1)
+		(exclude_from_sim no)
+		(in_bom yes)
+		(on_board yes)
+		(dnp no)
+		(fields_autoplaced yes)
+		(property "Reference" "U8"
+			(at -37.7189 100.33 0)
+			(effects
+				(font
+					(size 1.27 1.27)
+				)
+				(justify left)
+			)
+		)
+		(property "Value" "USBLC6-2SC6"
+			(at -37.7189 102.87 0)
+			(effects
+				(font
+					(size 1.27 1.27)
+				)
+				(justify left)
+			)
+		)
+		(property "Footprint" "Package_TO_SOT_SMD:SOT-23-6"
+			(at -38.1 114.3 0)
+			(effects
+				(font
+					(size 1.27 1.27)
+					(italic yes)
+				)
+				(justify left)
+				(hide yes)
+			)
+		)
+		(property "Datasheet" "https://www.st.com/resource/en/datasheet/usblc6-2.pdf"
+			(at -38.1 116.205 0)
+			(effects
+				(font
+					(size 1.27 1.27)
+				)
+				(justify left)
+				(hide yes)
+			)
+		)
+		(property "Description" "Very low capacitance ESD protection diode, 2 data-line, SOT-23-6"
+			(at -39.37 107.95 0)
+			(effects
+				(font
+					(size 1.27 1.27)
+				)
+				(hide yes)
+			)
+		)
+		(pin "5"
+		)
+		(pin "1"
+		)
+		(pin "3"
+		)
+		(pin "4"
+		)
+		(pin "2"
+		)
+		(pin "6"
+		)
+		(instances
+			(project ""
+				(path "/6f79ab9c-e294-456a-a1e3-a27257d9f14e"
+					(reference "U8")
+					(unit 1)
+				)
+			)
+		)
+	)
+	(symbol
 		(lib_id "Device:C")
 		(at 262.89 39.37 0)
@@
 			)
 		)
-		(property "Footprint" "Connector_PinHeader_2.54mm:PinHeader_1x04_P2.54mm_Vertical"
+		(property "Footprint" "AkiraBallParts:OLED_PinHeader_1x04_P2.54mm"
 			(at 129.54 170.18 0)
 			(effects

Commit message: Before routing PCB
Parts:
- removed U8: USBLC6-2SC6, Package_TO_SOT_SMD:SOT-23-6, symbol Power_Protection:USBLC6-2SC6
- added H1, H2, H3, H4, H5, H6, H7: MountingHole_Pad, AkiraBallParts:M2 Mounting Hole, symbol Mechanical:MountingHole_Pad
Connections:
- net GND: now also H1.1, H2.1, H3.1, H4.1, H5.1, H6.1, H7.1
Other:
- note added: "PMW 3360"
- moved on the sheet: C10, C11, R1_6, R1_7, R1_8, U3

Commit message: Dump
Parts:
- ISP1: renamed from J1; footprint Connector_PinHeader_2.54mm:PinHeader_2x03_P2.54mm_Vertical -> AkiraBallParts:SKEDD_6PinConnectingHole
- LS1: renamed from U4; JLCPCB Part # (none) -> C9382
- LS2: renamed from U5; JLCPCB Part # (none) -> C9382
- LS3: renamed from U6; JLCPCB Part # (none) -> C9382
- LS4: renamed from U7; JLCPCB Part # (none) -> C9382
- VR1: renamed from U2; JLCPCB Part # (none) -> C59200
- renumbered U1 to ATMEGA328P1, SW_V_1 to KNOB1, U3 to PMW3360, SW_R_1 to SCROLL_RING1, J2 to USB1
Connections:
- net CRYSTAL+: now reaches ATMEGA328P1.10 (PB7), C2.2, Y1.2
- net CRYSTAL-: now reaches ATMEGA328P1.9 (PB6), C1.2, Y1.1
Other:
- moved on the sheet: C1, C2, Y1

Commit message: Before PCB Fix
Connections:
- net +5V: now also LS3.5 (DIR)
- net NCS: no longer LS3.5 (DIR)
- net RING_A: no longer KNOB1.A
- net VK_A: now reaches ATMEGA328P1.24 (PC1)
- net VK_A: now also KNOB1.A
Other:
- note added: "Revision Notes: 1. - Connected Volume knob Pin A to Atmega328P Pin 24 - LS3 DIR was NCS. Fixed to be v5+"
Changed lines of the file:
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@@
 		)
 	)
+	(text "Revision Notes: \n1. \n- Connected Volume knob Pin A to Atmega328P Pin 24\n- LS3 DIR was NCS. Fixed to be v5+"
+		(exclude_from_sim no)
+		(at 345.948 211.074 0)
+		(effects
+			(font
+				(size 1.27 1.27)
+			)
+			(justify left)
+		)
+	)
 	(text "Buttons & Encoders"
 		(exclude_from_sim no)
@@
 	)
 	(junction
-		(at 31.75 59.69)
-		(diameter 0)
-		(color 0 0 0 0)
-	)
-	(junction
 		(at 198.12 34.29)
 		(diameter 0)
@@
 	(wire
 		(pts
-			(xy 30.48 63.5) (xy 31.75 63.5)
-		)
-		(stroke
-			(width 0)
-			(type default)
-		)
-	)
-	(wire
-		(pts
 			(xy 250.19 44.45) (xy 250.19 45.72)
 		)
@@
 	(wire
 		(pts
+			(xy 57.15 59.69) (xy 60.96 59.69)
+		)
+		(stroke
+			(width 0)
+			(type default)
+		)
+	)
+	(wire
+		(pts
 			(xy 111.76 29.21) (xy 101.6 29.21)
 		)
@@
 	(wire
 		(pts
-			(xy 60.96 59.69) (xy 31.75 59.69)
-		)
-		(stroke
-			(width 0)
-			(type default)
-		)
-	)
-	(wire
-		(pts
 			(xy 135.89 73.66) (xy 133.35 73.66)
 		)
@@
 	(wire
 		(pts
-			(xy 31.75 63.5) (xy 31.75 59.69)
-		)
-		(stroke
-			(width 0)
-			(type default)
-		)
-	)
-	(wire
-		(pts
 			(xy 125.73 92.71) (xy 125.73 73.66)
 		)
@@
 	(wire
 		(pts
-			(xy 31.75 59.69) (xy 30.48 59.69)
+			(xy 57.15 82.55) (xy 60.96 82.55)
 		)
 		(stroke
@@
 	(global_label "RING_A"
 		(shape input)
-		(at 30.48 63.5 180)
+		(at 57.15 59.69 180)
 		(effects
 			(font
@@
 		)
 		(property "Intersheetrefs" "${INTERSHEET_REFS}"
-			(at 30.48 63.5 0)
+			(at 57.15 59.69 0)
 			(effects
 				(font
@@
 		)
 	)
-	(global_label "NCS"
-		(shape input)
-		(at 307.34 101.6 180)
-		(effects
-			(font
-				(size 1.27 1.27)
-			)
-			(justify right)
-		)
-		(property "Intersheetrefs" "${INTERSHEET_REFS}"
-			(at 307.34 101.6 0)
-			(effects
-				(font
-					(size 1.27 1.27)
-				)
-				(hide yes)
-			)
-		)
-	)
 	(global_label "VK_A"
 		(shape input)
-		(at 30.48 59.69 180)
+		(at 57.15 82.55 180)
 		(effects
 			(font
@@
 		)
 		(property "Intersheetrefs" "${INTERSHEET_REFS}"
-			(at 30.48 59.69 0)
+			(at 57.15 82.55 0)
 			(effects
 				(font
@@
 					(unit 1)
 				)
+			)
+		)
+	)
+	(symbol
+		(lib_id "Akira_board-rescue:+5V-power")
+		(at 307.34 101.6 90)
+		(unit 1)
+		(exclude_from_sim no)
+		(in_bom yes)
+		(on_board yes)
+		(dnp no)
+		(property "Reference" "#PWR029"
+			(at 311.15 101.6 0)
+			(effects
+				(font
+					(size 1.27 1.27)
+				)
+				(hide yes)
+			)
+		)
+		(property "Value" "+5V"
+			(at 302.9458 101.219 0)
+			(effects
+				(font
+					(size 1.27 1.27)
+				)
+			)
+		)
+		(property "Footprint" ""
+			(at 307.34 101.6 0)
+			(effects
+				(font
+					(size 1.27 1.27)
+				)
+				(hide yes)
+			)
+		)
+		(property "Datasheet" ""
+			(at 307.34 101.6 0)
+			(effects
+				(font
+					(size 1.27 1.27)
+				)
+				(hide yes)
+			)
+		)
+		(property "Description" ""
+			(at 307.34 101.6 0)
+			(effects
+				(font
+					(size 1.27 1.27)
+				)
+				(hide yes)
+			)
+		)
+		(pin "1"
+		)
+		(instances
+			(project "Akira_board"
+				(path "/6f79ab9c-e294-456a-a1e3-a27257d9f14e"
+					(reference "#PWR029")
+					(unit 1)
+				)

Commit message: Save for now
Parts:
- removed C10: 4.7uF, Capacitor_THT:C_Rect_L4.0mm_W2.5mm_P2.50mm, symbol Akira_board-rescue:CP1-Device
- removed C3: 4.7uF, Capacitor_THT:CP_Radial_D4.0mm_P1.50mm, symbol Akira_board-rescue:CP1-Device
- removed SW1: Reset SW, Button_Switch_THT:SW_PUSH_6mm, symbol Switch:SW_Push
- removed SW2: Boot SW, Button_Switch_THT:SW_PUSH_6mm, symbol Switch:SW_Push
- removed Y1: 16MHz, Crystal:Crystal_HC49-4H_Vertical, symbol Device:Crystal
- added C10, C12: 4.7uF, Capacitor_SMD:C_0805_2012Metric, symbol Device:C
- added R1_10, R1_11, R1_9: 2R, Resistor_SMD:R_0603_1608Metric, symbol Device:R
- added R1_12, R1_13: 20R, Resistor_SMD:R_0603_1608Metric, symbol Device:R
- added R2, R5: 7.5K, Resistor_SMD:R_0603_1608Metric, symbol Device:R
- added U1, U2: ~, Akira_Ball_Parts:Switch SMD-4P,5.1x5.1mm, symbol Akira_Ball_Symbols:SMD-4P_Switch
- added Y2: Crystal_GND24, Crystal:Crystal_SMD_3225-4Pin_3.2x2.5mm, symbol Device:Crystal_GND24
- C1, C2: value 22p -> 12p; footprint Capacitor_THT:C_Rect_L4.0mm_W2.5mm_P2.50mm -> Capacitor_SMD:C_0603_1608Metric; JLCPCB Part # (none) -> C38523
- C11, C4, C5, C6, C8, C9: footprint Capacitor_THT:C_Disc_D3.8mm_W2.6mm_P2.50mm -> Capacitor_SMD:C_0603_1608Metric; JLCPCB Part # (none) -> C14663
- C7: footprint Capacitor_THT:C_Rect_L4.0mm_W2.5mm_P2.50mm -> Capacitor_SMD:C_0603_1608Metric; JLCPCB Part # (none) -> C15849
- D1, D2: footprint Diode_THT:D_DO-35_SOD27_P7.62mm_Horizontal -> Diode_SMD:D_SOD-123; JLCPCB Part # (none) -> C22395553
- D_I_1, D_I_2, D_I_3, D_I_4, D_I_5: footprint Diode_THT:D_DO-35_SOD27_P7.62mm_Horizontal -> Diode_SMD:D_SOD-123; JLCPCB Part # (none) -> C81598
- F1: footprint Fuse:Fuse_Bourns_MF-RG300 -> Fuse:Fuse_0805_2012Metric; JLCPCB Part # (none) -> C269102
- R1, R1_6, R1_8: footprint Resistor_THT:R_Axial_DIN0207_L6.3mm_D2.5mm_P7.62mm_Horizontal -> Resistor_SMD:R_0603_1608Metric; JLCPCB Part # (none) -> C25804; Wattage 1/2 -> 1/10
- R1_1, R1_2: footprint Resistor_THT:R_Axial_DIN0207_L6.3mm_D2.5mm_P7.62mm_Horizontal -> Resistor_SMD:R_0603_1608Metric; JLCPCB Part # (none) -> C23186; Wattage 1/2 -> 1/10
- R1_3, R1_4: value 75R -> 47R; footprint Resistor_THT:R_Axial_DIN0207_L6.3mm_D2.5mm_P7.62mm_Horizontal -> Resistor_SMD:R_0603_1608Metric; JLCPCB Part # (none) -> C23182; Wattage 1/2 -> 1/10
- R1_5: footprint Resistor_THT:R_Axial_DIN0207_L6.3mm_D2.5mm_P7.62mm_Horizontal -> Resistor_SMD:R_0603_1608Metric; JLCPCB Part # (none) -> C22843; Wattage 1/2 -> 1/10
- R1_7: value 39R -> 33R; footprint Resistor_THT:R_Axial_DIN0207_L6.3mm_D2.5mm_P7.62mm_Horizontal -> Resistor_SMD:R_0603_1608Metric; JLCPCB Part # (none) -> C23140; Wattage 1/2 -> 1/10
- R2_1, R2_2: footprint Resistor_THT:R_Axial_DIN0207_L6.3mm_D2.5mm_P7.62mm_Horizontal -> Resistor_SMD:R_0603_1608Metric; JLCPCB Part # (none) -> C23162; Wattage 1/2 -> 1/10
- R3: value 37.4K -> 30K; footprint Resistor_THT:R_Axial_DIN0207_L6.3mm_D2.5mm_P7.62mm_Horizontal -> Resistor_SMD:R_0603_1608Metric; JLCPCB Part # (none) -> C22984; Wattage 1/4 -> 1/10
- R4: value 63.4K -> 56K; footprint Resistor_THT:R_Axial_DIN0207_L6.3mm_D2.5mm_P7.62mm_Horizontal -> Resistor_SMD:R_0603_1608Metric; JLCPCB Part # (none) -> C23206; Wattage 1/4 -> 1/10
- SW_M_1_1, SW_M_1_2, SW_M_2_1, SW_M_2_2: footprint AkiraBallParts:GM8.0 -> Akira_Ball_Parts:GM8.0
Connections:
- net +5V: now also C10.1
- net BOOT: now also U2.1, U2.2
- net CRYSTAL+: now also Y2.1
- net CRYSTAL-: now also Y2.3
- net D+: now also R1_12.2; no longer R1_4.2
- net D-: now also R1_13.1; no longer R1_3.1
- net GND: now also C10.2, C12.2, R5.2, U1.3, U1.4, U2.3, U2.4, Y2.2, Y2.4; no longer R4.2
- net RESET: now also U1.1, U1.2
- net VDD: now also R1_10.1; no longer R1_7.1
- net at C8.2, R4.1, VR1.4 (FB): now also R2.2; no longer R3.2
- net at C11.1, PMW3360.3 (VDDPIX): now also C12.1
- new net: R1_12.1, R1_4.2
- new net: R1_13.2, R1_3.1
- new net: R1_10.2, R1_11.1
- new net: R2.1, R3.2
- new net: R4.2, R5.1
- new net: R1_11.2, R1_9.1
- new net: R1_7.1, R1_9.2
Other:
- note added: "ATmega328P circuit [SMT]"
- note added: "Boot & Reset Button [SMT]"
- note added: "OK"
- note added: "OLED Display [SMT]"
- note added: "PMW 3360 [SMT]"
- note added: "Power Noise [SMT]"
- note added: "Power Regulator [SMT]"
- note added: "Revision Notes: 1. - Connected Volume knob Pin A to Atmega328P Pin 24 - LS3 DIR was NCS. Fixed to be v5+ 2. SMT Replacements - USB-C Connector Circuits Updated"
- note added: "USB-C Connector [SMT]"
- note removed: "ATmega328P circuit"
- note removed: "Boot & Reset Button"
- note removed: "OLED Display"
- note removed: "PMW 3360"
- note removed: "Power Noise"
- note removed: "Power Regulator"
- note removed: "Revision Notes: 1. - Connected Volume knob Pin A to Atmega328P Pin 24 - LS3 DIR was NCS. Fixed to be v5+"
- note removed: "USB-C Connector"
- moved on the sheet: ATMEGA328P1, C1, C2, D1, D2, R1, R1_3, R1_4, R4

Commit message: SMT (done hopefully)
Parts:
- added H8, H9: MountingHole_Pad, AkiraBallParts:M2 Mounting Hole, symbol Mechanical:MountingHole_Pad
- added R6: 10K, Resistor_SMD:R_0603_1608Metric, symbol Device:R
- ATMEGA328P1, ISP1, SCROLL_RING1, SW_M_1_1, SW_M_1_2, SW_M_2_1, SW_M_2_2: now not fitted
- KNOB1: footprint Rotary_Encoder:RotaryEncoder_Alps_EC11E-Switch_Vertical_H20mm -> Akira_Ball_Parts:RotaryEncoder_Alps_EC11E-Switch_Vertical_H20mm; now not fitted
- PMW3360: footprint AkiraBallParts:PMW3360_1 -> Akira_Ball_Parts:PMW3360_2
- U1, U2: value ~ -> SW
- USB1: footprint Connector_USB:USB_C_Receptacle_GCT_USB4085 -> Akira_Ball_Parts:USB_C_16P_SMD_C3025063; JLCPCB Part # (none) -> C3025063
Connections:
- net +5V: now also R6.2
- net BOOT: now also R6.1
Other:
- moved on the sheet: R1, U1
